File: pcb/LTPS_A.kicad_pcb (KiCad board)
At the start: 4 copper layers, 120 x 100 mm, 93 parts, among them X1 R114665000, X2 2311768-2

Commit message: fixed license
Other:
- board text added: "LTPS Licensed under CERN-OHL-W v2 Version 1.1 - May 2023"
- board text removed: "LTPS May 2023 Version 1.1"
Changed lines of the file:
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@@
     )
   )
-  (gr_rect (start 85.852 72.898) (end 94.996 99.822) (layer "F.Mask") (width 0.2) (fill solid))
+  (gr_rect (start 85.852 66.898) (end 94.996 105.822) (layer "F.Mask") (width 0.2) (fill solid))
   (gr_rect (start 91.694 44.196) (end 110.49 41.148) (layer "F.Mask") (width 0.2) (fill solid))
   (gr_rect (start 84 37.5) (end 204 137.5) (layer "Edge.Cuts") (width 0.1) (fill none))
-  (gr_text "LTPS\nMay 2023\nVersion 1.1" (at 90.424 86.36 270) (layer "F.Cu")
+  (gr_text "LTPS\nLicensed under CERN-OHL-W v2\nVersion 1.1 - May 2023" (at 90.424 86.36 270) (layer "F.Cu")
     (effects (font (size 1.5 1.5) (thickness 0.3)))
   )
